File: hardware/window-blind/window-blind.kicad_pcb (KiCad board)
At the start: 2 copper layers, 91.4 x 81.3 mm, 32 parts, among them IC1 ATMEGA48PA-A, P1 CONN_02X05, SW1 UP, SW2 DN, SW3 END1, SW4 END2, U1 SP3485CN, U2 L298N, U3 LM78L05ACZ, Y1 16M

Commit message: Changes from 2016-05-02
Parts:
- W1, W2, W3, W4, W5, W6: footprint Connect:1pin -> Wire_Pads:SolderWirePad_single_1mmDrill
Changed lines of the file:
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@@
     )
-  )
-  (module Connect:1pin (layer F.Cu)
-    (at 208.28 124.46)
-    (descr "module 1 pin (ou trou mecanique de percage)")
-    (tags DEV)
-    (fp_text reference W1 (at 0 -3.048) (layer F.SilkS)
-      (effects (font (size 1 1) (thickness 0.15)))
-    )
-    (fp_text value A (at 0 2.794) (layer F.Fab)
-      (effects (font (size 1 1) (thickness 0.15)))
-    )
-    (fp_circle (center 0 0) (end 0 -2.286) (layer F.SilkS) (width 0.15))
-    (pad 1 thru_hole circle (at 0 0) (size 4.064 4.064) (drill 3.048) (layers *.Cu *.Mask F.SilkS)
-      (net 32 "Net-(U1-Pad6)"))
-  )
-  (module Connect:1pin (layer F.Cu)
-    (at 198.12 124.46)
-    (descr "module 1 pin (ou trou mecanique de percage)")
-    (tags DEV)
-    (fp_text reference W2 (at 0 -3.048) (layer F.SilkS)
-      (effects (font (size 1 1) (thickness 0.15)))
-    )
-    (fp_text value B (at 0 2.794) (layer F.Fab)
-      (effects (font (size 1 1) (thickness 0.15)))
-    )
-    (fp_circle (center 0 0) (end 0 -2.286) (layer F.SilkS) (width 0.15))
-    (pad 1 thru_hole circle (at 0 0) (size 4.064 4.064) (drill 3.048) (layers *.Cu *.Mask F.SilkS)
-      (net 31 "Net-(U1-Pad7)"))
-  )
-  (module Connect:1pin (layer F.Cu)
-    (at 187.96 58.42)
-    (descr "module 1 pin (ou trou mecanique de percage)")
-    (tags DEV)
-    (fp_text reference W3 (at 0 -3.048) (layer F.SilkS)
-      (effects (font (size 1 1) (thickness 0.15)))
-    )
-    (fp_text value +12V (at 0 2.794) (layer F.Fab)
-      (effects (font (size 1 1) (thickness 0.15)))
-    )
-    (fp_circle (center 0 0) (end 0 -2.286) (layer F.SilkS) (width 0.15))
-    (pad 1 thru_hole circle (at 0 0) (size 4.064 4.064) (drill 3.048) (layers *.Cu *.Mask F.SilkS)
-      (net 40 "Net-(C10-Pad1)"))
-  )
-  (module Connect:1pin (layer F.Cu)
-    (at 198.12 58.42)
-    (descr "module 1 pin (ou trou mecanique de percage)")
-    (tags DEV)
-    (fp_text reference W4 (at 0 -3.048) (layer F.SilkS)
-      (effects (font (size 1 1) (thickness 0.15)))
-    )
-    (fp_text value M+ (at 0 2.794) (layer F.Fab)
-      (effects (font (size 1 1) (thickness 0.15)))
-    )
-    (fp_circle (center 0 0) (end 0 -2.286) (layer F.SilkS) (width 0.15))
-    (pad 1 thru_hole circle (at 0 0) (size 4.064 4.064) (drill 3.048) (layers *.Cu *.Mask F.SilkS)
-      (net 4 "Net-(D1-Pad2)"))
-  )
-  (module Connect:1pin (layer F.Cu)
-    (at 208.28 58.42)
-    (descr "module 1 pin (ou trou mecanique de percage)")
-    (tags DEV)
-    (fp_text reference W5 (at 0 -3.048) (layer F.SilkS)
-      (effects (font (size 1 1) (thickness 0.15)))
-    )
-    (fp_text value M- (at 0 2.794) (layer F.Fab)
-      (effects (font (size 1 1) (thickness 0.15)))
-    )
-    (fp_circle (center 0 0) (end 0 -2.286) (layer F.SilkS) (width 0.15))
-    (pad 1 thru_hole circle (at 0 0) (size 4.064 4.064) (drill 3.048) (layers *.Cu *.Mask F.SilkS)
-      (net 5 "Net-(D3-Pad2)"))
-  )
-  (module Connect:1pin (layer F.Cu)
-    (at 218.44 58.42)
-    (descr "module 1 pin (ou trou mecanique de percage)")
-    (tags DEV)
-    (fp_text reference W6 (at 0 -3.048) (layer F.SilkS)
-      (effects (font (size 1 1) (thickness 0.15)))
-    )
-    (fp_text value GND (at 0 2.794) (layer F.Fab)
-      (effects (font (size 1 1) (thickness 0.15)))
-    )
-    (fp_circle (center 0 0) (end 0 -2.286) (layer F.SilkS) (width 0.15))
-    (pad 1 thru_hole circle (at 0 0) (size 4.064 4.064) (drill 3.048) (layers *.Cu *.Mask F.SilkS)
-      (net 2 GND))
   )
   (module Buttons_Switches_SMD:SW_SPST_B3S-1000 (layer B.Cu)
@@
     )
   )
+  (module Wire_Pads:SolderWirePad_single_1mmDrill (layer F.Cu)
+    (at 208.28 124.46)
+    (fp_text reference W1 (at 0 -3.81) (layer F.SilkS)
+      (effects (font (size 1 1) (thickness 0.15)))
+    )
+    (fp_text value A (at -1.905 3.175) (layer F.Fab)
+      (effects (font (size 1 1) (thickness 0.15)))
+    )
+    (pad 1 thru_hole circle (at 0 0) (size 2.49936 2.49936) (drill 1.00076) (layers *.Cu *.Mask F.SilkS)
+      (net 32 "Net-(U1-Pad6)"))
+  )
+  (module Wire_Pads:SolderWirePad_single_1mmDrill (layer F.Cu)
+    (at 198.12 124.46)
+    (fp_text reference W2 (at 0 -3.81) (layer F.SilkS)
+      (effects (font (size 1 1) (thickness 0.15)))
+    )
+    (fp_text value B (at -1.905 3.175) (layer F.Fab)
+      (effects (font (size 1 1) (thickness 0.15)))
+    )
+    (pad 1 thru_hole circle (at 0 0) (size 2.49936 2.49936) (drill 1.00076) (layers *.Cu *.Mask F.SilkS)
+      (net 31 "Net-(U1-Pad7)"))
+  )
+  (module Wire_Pads:SolderWirePad_single_1mmDrill (layer F.Cu)
+    (at 187.96 58.42)
+    (fp_text reference W3 (at 0 -3.81) (layer F.SilkS)
+      (effects (font (size 1 1) (thickness 0.15)))
+    )
+    (fp_text value +12V (at -1.905 3.175) (layer F.Fab)
+      (effects (font (size 1 1) (thickness 0.15)))
+    )
+    (pad 1 thru_hole circle (at 0 0) (size 2.49936 2.49936) (drill 1.00076) (layers *.Cu *.Mask F.SilkS)
+      (net 40 "Net-(C10-Pad1)"))
+  )
+  (module Wire_Pads:SolderWirePad_single_1mmDrill (layer F.Cu)
+    (at 198.12 58.42)
+    (fp_text reference W4 (at 0 -3.81) (layer F.SilkS)
+      (effects (font (size 1 1) (thickness 0.15)))
+    )
+    (fp_text value M+ (at -1.905 3.175) (layer F.Fab)
+      (effects (font (size 1 1) (thickness 0.15)))
+    )
+    (pad 1 thru_hole circle (at 0 0) (size 2.49936 2.49936) (drill 1.00076) (layers *.Cu *.Mask F.SilkS)
+      (net 4 "Net-(D1-Pad2)"))
+  )
+  (module Wire_Pads:SolderWirePad_single_1mmDrill (layer F.Cu)
+    (at 208.28 58.42)
+    (fp_text reference W5 (at 0 -3.81) (layer F.SilkS)
+      (effects (font (size 1 1) (thickness 0.15)))
+    )
+    (fp_text value M- (at -1.905 3.175) (layer F.Fab)
+      (effects (font (size 1 1) (thickness 0.15)))
+    )
+    (pad 1 thru_hole circle (at 0 0) (size 2.49936 2.49936) (drill 1.00076) (layers *.Cu *.Mask F.SilkS)
+      (net 5 "Net-(D3-Pad2)"))
+  )
+  (module Wire_Pads:SolderWirePad_single_1mmDrill (layer F.Cu)
+    (at 218.44 58.42)
+    (fp_text reference W6 (at 0 -3.81) (layer F.SilkS)
+      (effects (font (size 1 1) (thickness 0.15)))
+    )
+    (fp_text value GND (at -1.905 3.175) (layer F.Fab)
+      (effects (font (size 1 1) (thickness 0.15)))
+    )
+    (pad 1 thru_hole circle (at 0 0) (size 2.49936 2.49936) (drill 1.00076) (layers *.Cu *.Mask F.SilkS)
+      (net 2 GND))
+  )
   (gr_circle (center 147.32 127) (end 149.86 127) (layer Edge.Cuts) (width 0.15))
