File: hardware/window-blind/window-blind.sch (KiCad schematic (older format))
At the start: 32 parts, among them IC1 ATMEGA48PA-A, P1 CONN_02X05, SW1 UP, SW2 DN, SW3 END1, SW4 END2, U1 SP3485CN, U2 L298N, U3 LM78L05ACZ, Y1 16M

Commit message: Changes from 2016-05-02
Parts:
- W1, W2, W3, W4, W5, W6: footprint Connect:1pin -> Wire_Pads:SolderWirePad_single_1mmDrill
Changed lines of the file:
@@
 F 0 "W4" H 7500 2770 50  0000 C CNN
 F 1 "M+" H 7500 2700 50  0000 C CNN
-F 2 "Connect:1pin" H 7700 2500 50  0001 C CNN
+F 2 "Wire_Pads:SolderWirePad_single_1mmDrill" H 7700 2500 50  0001 C CNN
 F 3 "" H 7700 2500 50  0000 C CNN
 	1    7500 2500
@@
 F 0 "W5" H 7500 3070 50  0000 C CNN
 F 1 "M-" H 7500 3000 50  0000 C CNN
-F 2 "Connect:1pin" H 7700 2800 50  0001 C CNN
+F 2 "Wire_Pads:SolderWirePad_single_1mmDrill" H 7700 2800 50  0001 C CNN
 F 3 "" H 7700 2800 50  0000 C CNN
 	1    7500 2800
@@
 F 0 "W3" H 7500 2420 50  0000 C CNN
 F 1 "+12V" H 7500 2350 50  0000 C CNN
-F 2 "Connect:1pin" H 7700 2150 50  0001 C CNN
+F 2 "Wire_Pads:SolderWirePad_single_1mmDrill" H 7700 2150 50  0001 C CNN
 F 3 "" H 7700 2150 50  0000 C CNN
 	1    7500 2150
@@
 F 0 "W6" H 7500 3420 50  0000 C CNN
 F 1 "GND" H 7500 3350 50  0000 C CNN
-F 2 "Connect:1pin" H 7700 3150 50  0001 C CNN
+F 2 "Wire_Pads:SolderWirePad_single_1mmDrill" H 7700 3150 50  0001 C CNN
 F 3 "" H 7700 3150 50  0000 C CNN
 	1    7500 3150
@@
 F 0 "W1" H 6250 5120 50  0000 C CNN
 F 1 "A" H 6250 5050 50  0000 C CNN
-F 2 "Connect:1pin" H 6450 4850 50  0001 C CNN
+F 2 "Wire_Pads:SolderWirePad_single_1mmDrill" H 6450 4850 50  0001 C CNN
 F 3 "" H 6450 4850 50  0000 C CNN
 	1    6250 4850
@@
 F 0 "W2" H 6250 5320 50  0000 C CNN
 F 1 "B" H 6250 5250 50  0000 C CNN
-F 2 "Connect:1pin" H 6450 5050 50  0001 C CNN
+F 2 "Wire_Pads:SolderWirePad_single_1mmDrill" H 6450 5050 50  0001 C CNN
 F 3 "" H 6450 5050 50  0000 C CNN
 	1    6250 5050

Commit message: Changes from 2016-05-11
Parts:
- removed P1: CONN_02X05, Pin_Headers:Pin_Header_Straight_2x05, symbol CONN_02X05
- added P1: CONN_02X03, Pin_Headers:Pin_Header_Straight_2x03, symbol CONN_02X03
- added R3, R4, R5, R6: 10k, Resistors_SMD:R_1206_HandSoldering, symbol R
- D1, D2, D3, D4: footprint Diodes_SMD:DO-214AB_Handsoldering -> DO-214AA(SMB):DO-214AA(SMB)
Connections:
- net +5V: now also P1.2 (P2), R3.1, R4.1, R5.1, R6.1
- net GND: now also P1.6 (P6)
- net at IC1.1 ((PCINT19/OC2B/INT1)PD3): no longer SW1.2
- net at R2.1, U1.2 (~RE~), U1.3 (DE): now also IC1.32 ((PCINT18/INT0)PD2); no longer IC1.11 ((PCINT23/AIN1)PD7)
- net at IC1.14 ((PCINT2/OC1B/~SS~)PB2): now also SW1.2, R3.2
- net at IC1.15 ((PCINT3/OC2A/MOSI)PB3): now also P1.4 (P4)
- net at IC1.16 ((PCINT4/MISO)PB4): now also P1.1 (P1)
- net at IC1.17 ((PCINT5/SCK)PB5): now also P1.3 (P3)
- net at IC1.2 ((PCINT20/XCK/T0)PD4), SW3.2: now also R5.2
- net at IC1.29 ((PCINT14/~RESET~)PC6): now also P1.5 (P5)
- net at SW2.2: now also IC1.11 ((PCINT23/AIN1)PD7), R4.2; no longer IC1.32 ((PCINT18/INT0)PD2)
- net at IC1.9 ((PCINT21/OC0B/T1)PD5), SW4.2: now also R6.2
- no-connect marks 18 -> 17
Other:
- moved on the sheet: SW1, SW2, SW3, SW4
