File: hardware/rpi-rs485-shield/rpi-rs485-shield.kicad_pcb (KiCad board)
At the start: 2 copper layers, 23.4 x 22.9 mm, 8 parts, among them P1 CONN_01X06, U1 SP3485EN

Commit message: Changes from 2016-05-11
Other:
- board size 23.4 x 22.9 mm -> 23.4 x 23.6 mm
Changed lines of the file:
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@@
     (links 16)
     (no_connects 0)
-    (area 0 0 0 0)
+    (area 117.827667 86.759 144.422 115.295)
     (thickness 1.6)
     (drawings 8)
@@
   )
   (setup
-    (last_trace_width 1)
+    (last_trace_width 0.25)
     (user_trace_width 0.25)
     (user_trace_width 0.5)
@@
   (gr_line (start 144.272 88.392) (end 144.272 111.252) (angle 90) (layer Edge.Cuts) (width 0.15))
   (gr_line (start 120.904 88.392) (end 144.272 88.392) (angle 90) (layer Edge.Cuts) (width 0.15))
-  (gr_line (start 124.206 90.424) (end 124.206 92.964) (angle 90) (layer Edge.Cuts) (width 0.15))
-  (gr_line (start 122.936 91.694) (end 125.476 91.694) (angle 90) (layer Edge.Cuts) (width 0.15))
-  (gr_circle (center 124.206 91.694) (end 125.73 91.694) (layer Edge.Cuts) (width 0.15))
+  (gr_line (start 124.206 87.884) (end 124.206 90.424) (angle 90) (layer Edge.Cuts) (width 0.15))
+  (gr_line (start 122.936 89.154) (end 125.476 89.154) (angle 90) (layer Edge.Cuts) (width 0.15))
+  (gr_circle (center 124.206 89.154) (end 125.73 89.154) (layer Edge.Cuts) (width 0.15))
   (segment (start 121.412 99.06) (end 121.41169 89.416986) (width 0.5) (layer B.Cu) (net 1))
-  (segment (start 136.652 99.854) (end 137.636 100.838) (width 1) (layer B.Cu) (net 1) (status 800000))
+  (segment (start 136.652 99.854) (end 137.636 100.838) (width 1) (layer B.Cu) (net 1))
   (segment (start 136.652 90.17) (end 136.652 99.854) (width 1) (layer B.Cu) (net 1))
   (segment (start 135.636 89.154) (end 136.652 90.17) (width 1) (layer B.Cu) (net 1))
   (segment (start 121.66569 89.162986) (end 135.636 89.154) (width 1) (layer B.Cu) (net 1))
   (segment (start 121.41169 89.416986) (end 121.66569 89.162986) (width 0.5) (layer B.Cu) (net 1))
-  (segment (start 137.636 100.838) (end 137.636 101.568) (width 0.5) (layer B.Cu) (net 1) (status C00000))
-  (segment (start 137.636 101.568) (end 138.811 102.743) (width 1) (layer B.Cu) (net 1) (status C00000))
-  (segment (start 122.936 99.06) (end 121.412 99.06) (width 1) (layer B.Cu) (net 1) (status 400000))
-  (segment (start 121.412 109.22) (end 122.936 109.22) (width 0.5) (layer B.Cu) (net 1) (status 800000))
+  (segment (start 137.636 100.838) (end 137.636 101.568) (width 0.5) (layer B.Cu) (net 1))
+  (segment (start 137.636 101.568) (end 138.811 102.743) (width 1) (layer B.Cu) (net 1))
+  (segment (start 122.936 99.06) (end 121.412 99.06) (width 1) (layer B.Cu) (net 1))
+  (segment (start 121.412 109.22) (end 122.936 109.22) (width 0.5) (layer B.Cu) (net 1))
   (segment (start 121.412 99.314) (end 121.412 109.22) (width 0.5) (layer B.Cu) (net 1))
   (segment (start 121.412 99.06) (end 121.412 99.314) (width 0.5) (layer B.Cu) (net 1))
@@
   (segment (start 128.207 99.346) (end 128.81 99.949) (width 0.5) (layer B.Cu) (net 1))
   (segment (start 128.778 99.346) (end 128.81 99.314) (width 0.5) (layer B.Cu) (net 1))
-  (segment (start 133.636 100.838) (end 133.636 100.87) (width 1) (layer B.Cu) (net 2) (status C00000))
-  (segment (start 133.636 100.87) (end 134.366 101.6) (width 1) (layer B.Cu) (net 2) (status C00000))
-  (segment (start 134.366 101.6) (end 134.366 106.426) (width 1) (layer B.Cu) (net 2) (status 400000))
+  (segment (start 133.636 100.838) (end 133.636 100.87) (width 1) (layer B.Cu) (net 2))
+  (segment (start 133.636 100.87) (end 134.366 101.6) (width 1) (layer B.Cu) (net 2))
+  (segment (start 134.366 101.6) (end 134.366 106.426) (width 1) (layer B.Cu) (net 2))
   (segment (start 134.366 106.426) (end 134.493 106.553) (width 0.5) (layer B.Cu) (net 2))
-  (segment (start 134.493 106.553) (end 138.811 106.553) (width 1) (layer B.Cu) (net 2) (status 800000))
+  (segment (start 134.493 106.553) (end 138.811 106.553) (width 1) (layer B.Cu) (net 2))
   (segment (start 122.936 96.52) (end 133.604 96.52) (width 1) (layer B.Cu) (net 2))
   (segment (start 133.636 96.552) (end 133.636 100.838) (width 1) (layer B.Cu) (net 2))
@@
   (segment (start 130.651 106.553) (end 130.016 105.918) (width 0.5) (layer B.Cu) (net 6))
   (segment (start 130.016 105.918) (end 130.016 105.442) (width 0.5) (layer B.Cu) (net 6))
-  (segment (start 138.811 105.283) (end 140.081 105.283) (width 0.5) (layer B.Cu) (net 7) (status 400000))
-  (segment (start 140.208 92.71) (end 139.192 91.694) (width 1) (layer B.Cu) (net 7) (status 800000))
+  (segment (start 138.811 105.283) (end 140.081 105.283) (width 0.5) (layer B.Cu) (net 7))
+  (segment (start 140.208 92.71) (end 139.192 91.694) (width 1) (layer B.Cu) (net 7))
   (segment (start 140.208 105.156) (end 140.208 92.71) (width 1) (layer B.Cu) (net 7))
   (segment (start 140.081 105.283) (end 140.208 105.156) (width 0.5) (layer B.Cu) (net 7))
-  (segment (start 138.811 104.013) (end 136.017 104.013) (width 0.5) (layer B.Cu) (net 8) (status 400000))
-  (segment (start 135.636 93.218) (end 134.112 91.694) (width 0.5) (layer B.Cu) (net 8) (status 800000))
+  (segment (start 138.811 104.013) (end 136.017 104.013) (width 0.5) (layer B.Cu) (net 8))
+  (segment (start 135.636 93.218) (end 134.112 91.694) (width 0.5) (layer B.Cu) (net 8))
   (segment (start 135.636 103.632) (end 135.636 93.218) (width 0.5) (layer B.Cu) (net 8))
   (segment (start 136.017 104.013) (end 135.636 103.632) (width 0.5) (layer B.Cu) (net 8))
